Commit message: Fixed wrong file path

File: assets/xacro/ycb_orange/assets.xml.xacro (robot description, xacro)
@@ -1,4 +1,4 @@
 <?xml version="1.0"?>
-<!--mujoco xmlns:xacro="http://ros.org/wiki/xacro">
+<mujoco xmlns:xacro="http://ros.org/wiki/xacro">
     <xacro:macro name="ycb_orange_assets">
         <asset>
@@ -8,12 +8,3 @@
         </asset>
     </xacro:macro>
-</mujoco-->
-<mujoco xmlns:xacro="http://ros.org/wiki/xacro">
-    <xacro:macro name="ycb_orange_assets">
-        <asset>
-            <mesh file="/home/zklinger/Robocup/src/mujoco_ycb/assets/meshes/ycb_orange/model.obj" name="ycb_orange" scale="1.0 1.0 1.0"/>
-            <texture name="ycb_orange" file="/home/zklinger/Robocup/src/mujoco_ycb/assets/meshes/ycb_orange/texture_map.png" type="2d"/>
-            <material name="ycb_orange" texture="ycb_orange"/>
-        </asset>
-    </xacro:macro>
 </mujoco>
